File: st_adap/st_adap.kicad_pcb (KiCad board)
At the start: 2 copper layers, 29 x 24 mm, 5 parts, among them J1 Conn_02x07_Odd_Even, J2 Conn_01x05_Socket, J3 Conn_01x05_Socket, J4 Conn_01x05_Socket, J5 Conn_01x03_Socket

Commit message: Generate fabrication files
Parts:
- moved J1 3.40 mm to (207.9, 101.6)
- moved J5 1.22 mm to (201.5, 114.6)
- moved J4 0.73 mm to (218.6, 114.5)
Connections:
- net /GND renamed /GND2
Routing:
- net /T_VCP_TX: track 9.51 -> 14.2 mm
- net /GND2: track 29.1 -> 33.4 mm
- net /T_JTDO/T_SWO: track 17.6 -> 20.7 mm
- net /T_VCP_RX: track 9.03 -> 12.1 mm
- net /T_VCC: track 29.8 -> 32.6 mm
- net /T_JCLK/T_SWCLK: track 18.3 -> 20.8 mm
- net /GNDDETECT: track 6.26 -> 8.31 mm
- net /T_NRST: track 6.36 -> 7.77 mm
- net /GND1: track 7.32 -> 6.09 mm
- net /T_JRCLK: track 6.27 -> 7.49 mm
- net /T_JTDI/NC: track 6.37 -> 7.24 mm
- net /T_JTMS/T_SWDIO: track 21.6 -> 22.3 mm
Other:
- board text added: "SWCLK"
