File: st_adap/st_adap.kicad_sch (KiCad schematic)
At the start: 5 parts, among them J1 Conn_02x07_Odd_Even, J2 Conn_01x05_Socket, J3 Conn_01x05_Socket, J4 Conn_01x05_Socket, J5 Conn_01x03_Socket

Commit message: Generate fabrication files
Connections:
- net GND renamed GND2
Changed lines of the file:
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@@
     (effects (font (size 0.7 0.7)) (justify left bottom))
   )
-  (label "GND" (at 86.868 76.2 0) (fields_autoplaced)
+  (label "GND2" (at 86.868 76.2 0) (fields_autoplaced)
     (effects (font (size 0.7 0.7)) (justify left bottom))
   )

Commit message: Generate gerber files
Other:
- moved on the sheet: J1, J2, J3, J4, J5
