File: socadap/st_adap.kicad_sch (KiCad schematic)
At the start: 5 parts, among them J1 Conn_02x07_Odd_Even, J2 Conn_01x05_Socket, J3 Conn_01x05_Socket, J4 Conn_01x05_Socket, J5 Conn_01x03_Socket

Commit message: Socket 2x7
Parts:
- J1: footprint Connector_PinHeader_1.27mm:PinHeader_2x07_P1.27mm_Vertical_SMD -> Connector_PinSocket_1.27mm:PinSocket_2x07_P1.27mm_Vertical
Connections:
- net GND1: now also J1.6 (Pin_6); no longer J1.5 (Pin_5)
- net GND2: now also J1.8 (Pin_8); no longer J1.7 (Pin_7)
- net GNDDETECT: now also J1.12 (Pin_12); no longer J1.11 (Pin_11)
- net T_JCLK/T_SWCLK: now also J1.5 (Pin_5); no longer J1.6 (Pin_6)
- net T_JRCLK: now also J1.10 (Pin_10); no longer J1.9 (Pin_9)
- net T_JTDI/NC: now also J1.9 (Pin_9); no longer J1.10 (Pin_10)
- net T_JTDO/T_SWO: now also J1.7 (Pin_7); no longer J1.8 (Pin_8)
- net T_JTMS/T_SWDIO: now also J1.3 (Pin_3); no longer J1.4 (Pin_4)
- net T_NRST: now also J1.11 (Pin_11); no longer J1.12 (Pin_12)
- net T_VCC: now also J1.4 (Pin_4); no longer J1.3 (Pin_3)
- net T_VCP_RX: now also J1.14 (Pin_14); no longer J1.13 (Pin_13)
- net T_VCP_TX: now also J1.13 (Pin_13); no longer J1.14 (Pin_14)
Changed lines of the file:
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@@
+    (stroke (width 0) (type default))
+  )
+  (wire (pts (xy 76.2 69.85) (xy 83.82 69.85))
+    (stroke (width 0) (type default))
+  )
+  (wire (pts (xy 119.38 43.18) (xy 123.19 43.18))
+    (stroke (width 0) (type default))
+  )
+  (wire (pts (xy 107.95 50.8) (xy 123.19 50.8))
+    (stroke (width 0) (type default))
+  )
+  (wire (pts (xy 139.7 67.31) (xy 93.98 67.31))
+    (stroke (width 0) (type default))
+  )
+  (wire (pts (xy 119.38 43.18) (xy 119.38 69.85))
+    (stroke (width 0) (type default))
+  )
+  (wire (pts (xy 77.47 48.26) (xy 82.55 48.26))
+    (stroke (width 0) (type default))
+  )
+  (wire (pts (xy 82.55 48.26) (xy 82.55 67.31))
+    (stroke (width 0) (type default))
+  )
+  (wire (pts (xy 83.82 55.88) (xy 83.82 69.85))
+    (stroke (width 0) (type default))
+  )
+  (wire (pts (xy 139.7 64.77) (xy 120.65 64.77))
+    (stroke (width 0) (type default))
+  )
+  (wire (pts (xy 76.2 67.31) (xy 82.55 67.31))
+    (stroke (width 0) (type default))
+  )
+  (wire (pts (xy 118.11 45.72) (xy 123.19 45.72))
+    (stroke (width 0) (type default))
+  )
+  (wire (pts (xy 83.82 55.88) (xy 95.25 55.88))
     (stroke (width 0) (type default))
   )
@@
     (stroke (width 0) (type default))
   )
-  (wire (pts (xy 76.2 69.85) (xy 83.82 69.85))
-    (stroke (width 0) (type default))
-  )
-  (wire (pts (xy 119.38 43.18) (xy 123.19 43.18))
-    (stroke (width 0) (type default))
-  )
-  (wire (pts (xy 107.95 50.8) (xy 123.19 50.8))
-    (stroke (width 0) (type default))
-  )
-  (wire (pts (xy 139.7 67.31) (xy 93.98 67.31))
-    (stroke (width 0) (type default))
-  )
-  (wire (pts (xy 119.38 43.18) (xy 119.38 69.85))
-    (stroke (width 0) (type default))
-  )
-  (wire (pts (xy 77.47 48.26) (xy 82.55 48.26))
-    (stroke (width 0) (type default))
-  )
-  (wire (pts (xy 82.55 48.26) (xy 82.55 67.31))
-    (stroke (width 0) (type default))
-  )
-  (wire (pts (xy 83.82 55.88) (xy 83.82 69.85))
+  (wire (pts (xy 77.47 43.18) (xy 93.98 43.18))
+    (stroke (width 0) (type default))
+  )
+  (wire (pts (xy 92.71 74.93) (xy 139.7 74.93))
+    (stroke (width 0) (type default))
+  )
+  (wire (pts (xy 107.95 45.72) (xy 118.11 45.72))
+    (stroke (width 0) (type default))
+  )
+  (wire (pts (xy 107.95 43.18) (xy 119.38 43.18))
+    (stroke (width 0) (type default))
+  )
+  (wire (pts (xy 77.47 45.72) (xy 95.25 45.72))
     (stroke (width 0) (type default))
   )
@@
     (stroke (width 0) (type default))
   )
-  (wire (pts (xy 139.7 64.77) (xy 120.65 64.77))
-    (stroke (width 0) (type default))
-  )
-  (wire (pts (xy 77.47 43.18) (xy 93.98 43.18))
-    (stroke (width 0) (type default))
-  )
-  (wire (pts (xy 76.2 67.31) (xy 82.55 67.31))
-    (stroke (width 0) (type default))
-  )
-  (wire (pts (xy 118.11 45.72) (xy 123.19 45.72))
-    (stroke (width 0) (type default))
-  )
-  (wire (pts (xy 83.82 55.88) (xy 95.25 55.88))
-    (stroke (width 0) (type default))
-  )
-  (wire (pts (xy 92.71 74.93) (xy 139.7 74.93))
-    (stroke (width 0) (type default))
-  )
-  (wire (pts (xy 107.95 45.72) (xy 118.11 45.72))
-    (stroke (width 0) (type default))
-  )
-  (wire (pts (xy 107.95 43.18) (xy 119.38 43.18))
-    (stroke (width 0) (type default))
-  )
   (wire (pts (xy 118.11 45.72) (xy 118.11 72.39))
     (stroke (width 0) (type default))
@@
   )
   (wire (pts (xy 107.95 55.88) (xy 115.57 55.88))
-    (stroke (width 0) (type default))
-  )
-  (wire (pts (xy 77.47 45.72) (xy 95.25 45.72))
     (stroke (width 0) (type default))
   )
@@
     )
   )
-  (symbol (lib_id "Connector_Generic:Conn_02x07_Odd_Even") (at 100.33 48.26 0) (unit 1)
-    (in_bom yes) (on_board yes) (dnp no) (fields_autoplaced)
+  (symbol (lib_id "Connector_Generic:Conn_02x07_Odd_Even") (at 102.87 48.26 0) (mirror y) (unit 1)
+    (in_bom yes) (on_board yes) (dnp no)
     (property "Reference" "J1" (at 101.6 34.925 0)
       (effects (font (size 1.27 1.27)))
@@
       (effects (font (size 1.27 1.27)))
     )
-    (property "Footprint" "Connector_PinHeader_1.27mm:PinHeader_2x07_P1.27mm_Vertical_SMD" (at 100.33 48.26 0)
-      (effects (font (size 1.27 1.27)) hide)
-    )
-    (property "Datasheet" "~" (at 100.33 48.26 0)
-      (effects (font (size 1.27 1.27)) hide)
-    )
-    (property "JLC#" "C2881912" (at 100.33 48.26 0)
-      (effects (font (size 1.27 1.27)) hide)
-    )
+    (property "Footprint" "Connector_PinSocket_1.27mm:PinSocket_2x07_P1.27mm_Vertical" (at 102.87 48.26 0)
+      (effects (font (size 1.27 1.27)) hide)
+    )
+    (property "Datasheet" "~" (at 102.87 48.26 0)
+      (effects (font (size 1.27 1.27)) hide)
+    )
+    (property "JLC#" "C2881912" (at 102.87 48.26 0)
+      (effects (font (size 1.27 1.27)) hide)
+    )

Commit message: Gen socadp
Parts:
- J1: JLC# C2881912 -> C5160804
Changed lines of the file:
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@@
       (effects (font (size 1.27 1.27)) hide)
     )
-    (property "JLC#" "C2881912" (at 102.87 48.26 0)
+    (property "JLC#" "C5160804" (at 102.87 48.26 0)
       (effects (font (size 1.27 1.27)) hide)
     )
